File: Light/Light.kicad_pcb (KiCad board)
At the start: 2 copper layers, 40 parts

Commit message: general board shape with screw mounting holes
Parts:
- moved H4 60.8 mm to (242.9, 15.0)
- moved H3 54.5 mm to (65.1, 15.0)
Other:
- board outline added: 308 x 22 mm
Changed lines of the file:
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@@
 	(footprint "MountingHole:MountingHole_6.4mm_M6"
 		(layer "F.Cu")
-		(at 114.5 38)
+		(at 65.1 15)
 		(descr "Mounting Hole 6.4mm, M6, no annular, generated by kicad-footprint-generator mountinghole.py")
 		(tags "mountinghole M6")
@@
 	(footprint "MountingHole:MountingHole_6.4mm_M6"
 		(layer "F.Cu")
-		(at 185.5 35)
+		(at 242.9 15)
 		(descr "Mounting Hole 6.4mm, M6, no annular, generated by kicad-footprint-generator mountinghole.py")
 		(tags "mountinghole M6")
@@
 		)
 	)
+	(gr_rect
+		(start -0.5 0)
+		(end 307.5 22)
+		(stroke
+			(width 0.05)
+			(type default)
+		)
+		(fill no)
+		(layer "Edge.Cuts")
+	)
 	(embedded_fonts no)

Commit message: general placement and first pass at routing
Parts:
- moved LED22 184.4 mm to (277.5, 4.00), turned to 180 degrees
- moved R8 183.1 mm to (277.0, 16.0), turned to 90 degrees
- moved LED23 180.2 mm to (290.5, 11.0), turned to 180 degrees
- moved LED24 178.1 mm to (303.5, 18.0), turned to 180 degrees
- moved LED19 149.9 mm to (238.5, 4.00), turned to 180 degrees
- moved LED20 144.4 mm to (251.5, 11.0), turned to 180 degrees
- moved LED21 142.1 mm to (264.5, 18.0), turned to 180 degrees
- moved R7 142.1 mm to (233.0, 16.0), turned to 90 degrees
- moved LED2 141.9 mm to (17.5, 11.0), turned to 180 degrees
- moved LED3 139.8 mm to (30.5, 18.0), turned to 180 degrees
- moved LED1 139.6 mm to (4.50, 4.00), turned to 180 degrees
- moved R1 126.9 mm to (4.00, 16.0), turned to 90 degrees
- moved LED16 117.7 mm to (199.5, 4.00), turned to 180 degrees
- moved R6 112.4 mm to (199.0, 16.0), turned to 90 degrees
- moved LED17 112.1 mm to (212.5, 11.0), turned to 180 degrees
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Connections:
- LED14 pad 2: Net-(LED14-Pad2) -> Net-(LED13-Pad1)
- LED15 pad 1: Net-(LED15-Pad1) -> GND
- LED15 pad 2: Net-(LED15-Pad2) -> Net-(LED14-Pad1)
- LED17 pad 2: Net-(LED13-Pad1) -> Net-(LED16-Pad1)
- LED18 pad 1: Net-(LED18-Pad1) -> GND
- LED18 pad 2: Net-(LED14-Pad1) -> Net-(LED17-Pad1)
- LED19 pad 2: Net-(LED15-Pad1) -> Net-(LED19-Pad2)
- LED20 pad 2: Net-(LED16-Pad1) -> Net-(LED19-Pad1)
- LED21 pad 2: Net-(LED17-Pad1) -> Net-(LED20-Pad1)
- LED22 pad 1: GND -> Net-(LED22-Pad1)
- LED22 pad 2: Net-(LED18-Pad1) -> Net-(LED22-Pad2)
- LED23 pad 1: GND -> Net-(LED23-Pad1)
- LED23 pad 2: Net-(LED19-Pad1) -> Net-(LED22-Pad1)
- LED24 pad 2: Net-(LED20-Pad1) -> Net-(LED23-Pad1)
- R6 pad 2: Net-(LED14-Pad2) -> Net-(LED16-Pad2)
- R7 pad 2: Net-(LED15-Pad2) -> Net-(LED19-Pad2)
- R8 pad 2: Net-(LED16-Pad2) -> Net-(LED22-Pad2)
Routing:
- net Net-(LED5-Pad1): track 0.00 -> 29.4 mm
- net Net-(LED8-Pad1): track 0.00 -> 17.1 mm
- net Net-(LED16-Pad1): track 0.00 -> 17.1 mm
- net Net-(LED22-Pad1): track 0.00 -> 16.5 mm
- net Net-(LED4-Pad1): track 0.00 -> 16.5 mm
- net Net-(LED7-Pad1): track 0.00 -> 16.5 mm
- net Net-(LED14-Pad1): track 0.00 -> 16.5 mm
- net Net-(LED13-Pad1): track 0.00 -> 16.5 mm
- net Net-(LED10-Pad1): track 0.00 -> 16.5 mm
- net Net-(LED1-Pad1): track 0.00 -> 16.2 mm
- net Net-(LED23-Pad1): track 0.00 -> 15.9 mm
- net Net-(LED20-Pad1): track 0.00 -> 15.9 mm
- net Net-(LED17-Pad1): track 0.00 -> 15.9 mm
- net Net-(LED11-Pad1): track 0.00 -> 15.9 mm
- net Net-(LED19-Pad1): track 0.00 -> 15.3 mm
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- added copper zone on F.Cu, net /V_Vehicle
- added copper zone on B.Cu, net GND
- added copper zone on F.Cu, net GND
Other:
- board size 308 x 22 mm -> 308 x 24 mm
